Commit message: Add plugin.

File: quadrotor_description/urdf/quadrotor.gazebo.xacro (robot description, xacro)
@@ -2,4 +2,9 @@
 <robot name="quadrotor" xmlns:xacro="http://www.ros.org/wiki/xacro">
     <xacro:include filename="$(find quadrotor_description)/urdf/quadrotor.urdf.xacro"/>
-    <!--    <xacro:include filename="$(find quadrotor_description)/urdf/quadrotor_plugins.gazebo.xacro" />-->
+    <gazebo>
+        <plugin name="gazebo_ros_control" filename="libquadrotor_hw_sim.so">
+            <robotNamespace>/</robotNamespace>
+            <robotSimType>quadrotor_gazebo/QuadrotorHWSim</robotSimType>
+        </plugin>
+    </gazebo>
 </robot>

File: quadrotor_description/urdf/quadrotor_base.urdf.xacro (robot description, xacro)
@@ -1,6 +1,6 @@
 <?xml version="1.0"?>
 <robot xmlns:xacro="http://www.ros.org/wiki/xacro">
-    <xacro:include filename="$(find quadrotor_description)/urdf/sensors/sonar_sensor.urdf.xacro"/>
-    <xacro:property name="pi" value="3.1415926535897931"/>
+    <!--    <xacro:include filename="$(find quadrotor_description)/urdf/sensors/sonar_sensor.urdf.xacro"/>-->
+    <!--    <xacro:property name="pi" value="3.1415926535897931"/>-->
     <!-- Main quadrotor link -->
     <xacro:macro name="quadrotor_base_macro">
